File: ThermalControl/ThermalControl v1.0/ThermalControl.kicad_sch (KiCad schematic)
At the start: 18 parts, among them J3 DC-005, J4 TEC, J6 COOLER, Q1 IRF540N, U1 NODE_MCU

Commit message: schematic versions
Connections:
- net at R4.1: now also C_LED1.1 (K); no longer C_LED1.2 (A)
- net at P_LED1.1 (K): now also R5.1; no longer U1.30 (D0)
- net at P_LED1.2 (A): now also U1.30 (D0); no longer R5.1
- net at U1.29 (D1): now also C_LED1.2 (A); no longer C_LED1.1 (K)
Other:
- moved on the sheet: C_LED1, P_LED1
Changed lines of the file:
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@@
     (pin "2")
   )
-  (symbol (lib_id "Device:LED") (at 152.4 83.82 0) (unit 1)
-    (in_bom yes) (on_board yes) (fields_autoplaced)
-    (property "Reference" "P_LED1" (id 0) (at 150.8125 77.47 0))
-    (property "Value" "LED" (id 1) (at 150.8125 80.01 0))
+  (symbol (lib_id "Device:LED") (at 152.4 83.82 180) (unit 1)
+    (in_bom yes) (on_board yes) (fields_autoplaced)
+    (property "Reference" "P_LED1" (id 0) (at 153.9875 76.2 0))
+    (property "Value" "LED" (id 1) (at 153.9875 78.74 0))
     (property "Footprint" "LED_THT:LED_D5.0mm" (id 2) (at 152.4 83.82 0)
       (effects (font (size 1.27 1.27)) hide)
@@
     (pin "2")
   )
-  (symbol (lib_id "Device:LED") (at 152.4 72.39 0) (unit 1)
-    (in_bom yes) (on_board yes) (fields_autoplaced)
-    (property "Reference" "C_LED1" (id 0) (at 150.8125 66.04 0))
-    (property "Value" "LED" (id 1) (at 150.8125 68.58 0))
+  (symbol (lib_id "Device:LED") (at 152.4 72.39 180) (unit 1)
+    (in_bom yes) (on_board yes) (fields_autoplaced)
+    (property "Reference" "C_LED1" (id 0) (at 153.9875 64.77 0))
+    (property "Value" "LED" (id 1) (at 153.9875 67.31 0))
     (property "Footprint" "LED_THT:LED_D5.0mm" (id 2) (at 152.4 72.39 0)
       (effects (font (size 1.27 1.27)) hide)
